File: businesscard.kicad_sch (KiCad schematic)
At the start: 6 parts

Commit message: stuff
Parts:
- added D1, D2, D3, D4: LED, symbol Device:LED
- added R1: R, symbol Device:R
- renumbered 11 to L1
Connections:
- net SCL: now reaches U2.11 (PIO0_4/SCL)
- net SDA: now reaches U2.12 (PIO0_5/SDA)
- net LEDC4: now reaches U2.13 (PIO0_7/CT16B_M1)
- net LEDC4: now also D4.1 (K)
- net LEDR1: now reaches U2.2 (PIO0_1/CLKOUT)
- net LEDR1: now also R1.1
- net LEDC1: now reaches U2.4 (PIO0_6/SCLK)
- net LEDC1: now also D1.1 (K)
- net LEDC2: now reaches U2.5 (PIO0_8/MISO)
- net LEDC2: now also D2.1 (K)
- net LEDC3: now reaches U2.6 (PIO0_9/MOSI)
- net LEDC3: now also D3.1 (K)
- new net: D1.2 (A), D2.2 (A), D3.2 (A), D4.2 (A), R1.2
Other:
- moved on the sheet: C2, C3, C4
