File: businesscard.kicad_sch (KiCad schematic)
At the start: 11 parts

Commit message: update schematics and stuff
Parts:
- added J1: Conn_01x08_Pin, Library:8-Pin-Pads, symbol Connector:Conn_01x08_Pin
- D1, D2, D3, D4: footprint (none) -> LED_SMD:LED_0805_2012Metric
- R1: footprint (none) -> Resistor_SMD:R_0201_0603Metric
Connections:
- net GND: now also J1.2 (Pin_2)
- net SCL: now also J1.8 (Pin_8)
- net SDA: now also J1.7 (Pin_7)
- net SWCLK: now reaches U2.15 (PIO0_10/CT32B_M0/SWCLK)
- net SWCLK: now also J1.4 (Pin_4)
- net SWDIO: now reaches U2.16 (PIO0_11/CT32B_M1/SWDIO)
- net SWDIO: now also J1.3 (Pin_3)
- net VCC: now reaches C2.1, U2.7 (VDDBAT)
- net VCC: now also J1.1 (Pin_1), J1.6 (Pin_6)
- net RESET: now reaches C3.1, U2.9 (RESETN)
- net RESET: now also J1.5 (Pin_5)

Commit message: finish pcb routing
Parts:
- removed D4: LED, LED_SMD:LED_0805_2012Metric, symbol Device:LED
Connections:
- net RESET: now also J1.3 (Pin_3); no longer J1.5 (Pin_5)
- net SWDIO: now also J1.5 (Pin_5); no longer J1.3 (Pin_3)
- net VCC: no longer J1.6 (Pin_6)
- net WAKE: now reaches C4.1, U2.1 (PIO0_0/WAKEUP)
- net WAKE: now also J1.6 (Pin_6)
- net at C1.2, U2.19 (LB): now also L1.2; no longer L1.P$2
- net at C1.1, U2.20 (LA): now also L1.1; no longer L1.P$1
- net LEDC4: no longer names the net of U2.13 (PIO0_7/CT16B_M1)
Other:
- moved on the sheet: C1, L1
Changed lines of the file:
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@@
-	)
-	(junction
-		(at 152.4 127)
-		(diameter 0)
-		(color 0 0 0 0)
 	)
 	(junction
@@
 	)
 	(junction
-		(at 204.47 81.28)
-		(diameter 0)
-		(color 0 0 0 0)
-	)
-	(junction
 		(at 91.44 85.09)
 		(diameter 0)
@@
 	)
 	(junction
-		(at 204.47 88.9)
+		(at 203.2 88.9)
 		(diameter 0)
 		(color 0 0 0 0)
 	)
+	(junction
+		(at 203.2 81.28)
+		(diameter 0)
+		(color 0 0 0 0)
+	)
 	(wire
 		(pts
@@
 	(wire
 		(pts
+			(xy 203.2 88.9) (xy 208.28 88.9)
+		)
+		(stroke
+			(width 0)
+			(type default)
+		)
+	)
+	(wire
+		(pts
 			(xy 139.7 127) (xy 152.4 127)
 		)
@@
 	(wire
 		(pts
-			(xy 208.28 92.71) (xy 213.36 92.71)
-		)
-		(stroke
-			(width 0)
-			(type default)
-		)
-	)
-	(wire
-		(pts
-			(xy 165.1 127) (xy 165.1 130.81)
+			(xy 208.28 92.71) (xy 214.63 92.71)
 		)
 		(stroke
@@
 	(wire
 		(pts
-			(xy 199.39 81.28) (xy 204.47 81.28)
-		)
-		(stroke
-			(width 0)
-			(type default)
-		)
-	)
-	(wire
-		(pts
-			(xy 204.47 88.9) (xy 208.28 88.9)
+			(xy 199.39 81.28) (xy 203.2 81.28)
 		)
 		(stroke
@@
 	(wire
 		(pts
+			(xy 203.2 81.28) (xy 208.28 81.28)
+		)
+		(stroke
+			(width 0)
+			(type default)
+		)
+	)
+	(wire
+		(pts
 			(xy 189.23 83.82) (xy 199.39 83.82)
 		)
@@
 	(wire
 		(pts
-			(xy 204.47 81.28) (xy 208.28 81.28)
-		)
-		(stroke
-			(width 0)
-			(type default)
-		)
-	)
-	(wire
-		(pts
 			(xy 189.23 86.36) (xy 199.39 86.36)
 		)
@@
 	(wire
 		(pts
-			(xy 152.4 127) (xy 165.1 127)
-		)
-		(stroke
-			(width 0)
-			(type default)
-		)
-	)
-	(wire
-		(pts
 			(xy 208.28 81.28) (xy 208.28 77.47)
 		)
@@
 	(wire
 		(pts
-			(xy 199.39 88.9) (xy 204.47 88.9)
+			(xy 199.39 88.9) (xy 203.2 88.9)
 		)
 		(stroke
@@
 	(wire
 		(pts
-			(xy 208.28 77.47) (xy 213.36 77.47)
+			(xy 208.28 77.47) (xy 214.63 77.47)
 		)
 		(stroke
@@
 		)
 	)
-	(label "SWDIO"
-		(at 83.82 120.65 270)
-		(effects
-			(font
-				(size 1.27 1.27)
-			)
-			(justify right bottom)
-		)
-	)
 	(label "SDA"
 		(at 115.57 97.79 180)
@@
 		)
 	)
-	(label "VDDBAT"
-		(at 76.2 120.65 270)
-		(effects
-			(font
-				(size 1.27 1.27)
-			)
-			(justify right bottom)
-		)
-	)
 	(label "LEDC3"
 		(at 115.57 82.55 180)
@@
 		)
 	)
-	(label "LEDC4"
-		(at 115.57 100.33 180)
+	(label "SWDIO"
+		(at 78.74 120.65 270)
 		(effects
 			(font
@@
 		)
 	)
+	(label "WAKE"
+		(at 76.2 120.65 270)
+		(effects
+			(font
+				(size 1.27 1.27)
+			)
+			(justify right bottom)
+		)
+	)
 	(label "SWDIO"
 		(at 189.23 93.98 0)
@@
 		)
 	)
+	(label "RESET"
+		(at 83.82 120.65 270)
+		(effects
+			(font
+				(size 1.27 1.27)
+			)
+			(justify right bottom)
+		)
+	)
 	(label "LEDC2"
 		(at 139.7 138.43 270)
@@
 		)
 	)
+	(label "SWCLK"
+		(at 81.28 120.65 270)
+		(effects
+			(font
+				(size 1.27 1.27)
+			)
+			(justify right bottom)
+		)
+	)
 	(label "LEDC1"
 		(at 127 138.43 270)
@@
 		)
 	)
-	(label "LEDC4"
-		(at 165.1 138.43 270)
-		(effects
-			(font
-				(size 1.27 1.27)
-			)
-			(justify right bottom)
-		)
-	)
 	(label "SWCLK"
 		(at 189.23 96.52 0)
@@
 		)
 	)
+	(label "WAKE"
+		(at 114.3 68.58 180)
+		(effects
+			(font
+				(size 1.27 1.27)
+			)
+			(justify right bottom)
+		)
+	)
 	(label "LEDR1"
 		(at 114.3 127 180)
-		(effects
-			(font
-				(size 1.27 1.27)
-			)
-			(justify right bottom)
-		)
-	)
-	(label "SWCLK"
-		(at 81.28 120.65 270)
-		(effects
-			(font
-				(size 1.27 1.27)
-			)
-			(justify right bottom)
-		)
-	)
-	(label "RESET"
-		(at 78.74 120.65 270)
 		(effects
 			(font
@@
 	)
 	(symbol
-		(lib_id "Device:LED")
-		(at 165.1 134.62 90)
-		(unit 1)
-		(exclude_from_sim no)
-		(in_bom yes)
-		(on_board yes)
-		(dnp no)
-		(fields_autoplaced yes)
-		(property "Reference" "D4"
-			(at 168.91 134.9374 90)
-			(effects
-				(font
-					(size 1.27 1.27)
-				)
-				(justify right)
-			)
-		)
-		(property "Value" "LED"
-			(at 168.91 137.4774 90)
-			(effects
-				(font
-					(size 1.27 1.27)
-				)
-				(justify right)
-			)
-		)
-		(property "Footprint" "LED_SMD:LED_0805_2012Metric"
-			(at 165.1 134.62 0)
-			(effects
-				(font
-					(size 1.27 1.27)
-				)
-				(hide yes)
-			)
-		)
-		(property "Datasheet" "~"
-			(at 165.1 134.62 0)
-			(effects
-				(font
-					(size 1.27 1.27)
-				)
-				(hide yes)
-			)
-		)
-		(property "Description" "Light emitting diode"
-			(at 165.1 134.62 0)
-			(effects
-				(font
-					(size 1.27 1.27)
-				)
-				(hide yes)
-			)
-		)
-		(property "Sim.Pins" "1=K 2=A"
-			(at 165.1 134.62 0)
-			(effects
-				(font
-					(size 1.27 1.27)
-				)
-				(hide yes)
-			)
-		)
-		(pin "1"
-		)
-		(pin "2"
-		)
-		(instances
-			(project "businesscard"
-				(path "/57f92133-e803-40c7-8f5f-2b073fd15cf8"
-					(reference "D4")
-					(unit 1)
-				)
-			)
-		)
-	)
-	(symbol
 		(lib_id "power:GND")
 		(at 115.57 87.63 270)
@@
 	(symbol
 		(lib_id "Device:C")
-		(at 204.47 85.09 0)
+		(at 203.2 85.09 0)
 		(unit 1)
 		(exclude_from_sim no)
@@
 		(fields_autoplaced yes)
 		(property "Reference" "C1"
-			(at 208.28 83.8199 0)
+			(at 207.01 83.8199 0)
 			(effects
 				(font
@@
 		)
 		(property "Value" "1.2pF"
-			(at 208.28 86.3599 0)
+			(at 207.01 86.3599 0)
 			(effects
 				(font
@@
 		)
 		(property "Footprint" "Capacitor_SMD:C_0201_0603Metric"
-			(at 205.4352 88.9 0)
+			(at 204.1652 88.9 0)
 			(effects
 				(font
@@
 		)
 		(property "Datasheet" "~"
-			(at 204.47 85.09 0)
+			(at 203.2 85.09 0)
 			(effects
 				(font
@@
 		)
 		(property "Description" "Unpolarized capacitor"
-			(at 204.47 85.09 0)
+			(at 203.2 85.09 0)
 			(effects
 				(font
@@
 		)
 		(instances
-			(project ""
+			(project "businesscard"
 				(path "/57f92133-e803-40c7-8f5f-2b073fd15cf8"
 					(reference "C1")
@@
 	(symbol
 		(lib_id "25X48MM_NFC_ANTENNA:25X48MM_NFC_ANTENNA")
-		(at 213.36 85.09 0)
+		(at 214.63 85.09 0)
 		(unit 1)
 		(exclude_from_sim no)
@@
 		(fields_autoplaced yes)
 		(property "Reference" "L1"
-			(at 215.9 84.4549 0)
+			(at 217.17 84.4549 0)
 			(effects
 				(font
@@
 		)
 		(property "Value" "~"
-			(at 215.9 86.36 0)
+			(at 217.17 86.36 0)
 			(effects
 				(font
@@
 		)
 		(property "Footprint" "Library:25X48MM_NFC_EXPOSED_ANTENNA"
-			(at 213.36 85.09 0)
+			(at 214.63 85.09 0)
 			(effects
 				(font
@@
 		)
 		(property "Datasheet" ""
-			(at 213.36 85.09 0)
+			(at 214.63 85.09 0)
 			(effects
 				(font
@@
 		)
 		(property "Description" ""
-			(at 213.36 85.09 0)
-			(effects
-				(font
-					(size 1.27 1.27)
-				)
-				(hide yes)
-			)
-		)
-		(pin "P$2"
-		)
-		(pin "P$1"
+			(at 214.63 85.09 0)
+			(effects
+				(font
+					(size 1.27 1.27)
+				)
+				(hide yes)
+			)
+		)
+		(pin "1"
+		)
+		(pin "2"
 		)
 		(instances

Commit message: finalize pcb
Parts:
- R1: value R -> 330
Changed lines of the file:
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@@
 			)
 		)
-		(property "Value" "R"
+		(property "Value" "330"
 			(at 118.11 123.19 90)
 			(effects

Commit message: business card stuff
Parts:
- added H1: HoldingHole, Library:HoldingHole, symbol Mechanical:MountingHole_Pad
- C2, C3, C4: footprint Capacitor_SMD:C_0201_0603Metric -> Capacitor_SMD:C_0402_1005Metric
- D1, D2, D3: footprint LED_SMD:LED_0805_2012Metric -> LED_SMD:LED_1206_3216Metric
- R1: footprint Resistor_SMD:R_0201_0603Metric -> Resistor_SMD:R_0402_1005Metric
Connections:
- net GND: now also H1.1
- net LEDC1: now also U2.6 (PIO0_9/MOSI); no longer U2.4 (PIO0_6/SCLK)
- net LEDC3: now also U2.4 (PIO0_6/SCLK); no longer U2.6 (PIO0_9/MOSI)
