File: businesscard.kicad_pcb (KiCad board)
At the start: 2 copper layers, 88.9 x 50.8 mm, 6 parts

Commit message: stuff
Parts:
- moved C4 4.75 mm to (154.5, 90.5), turned to 90 degrees
- moved C3 4.20 mm to (149.7, 93.9), turned to 180 degrees
- moved C2 4.10 mm to (149.9, 92.7)
- moved U2 3.40 mm to (153.2, 94.2)
- moved C1 1.54 mm to (157.0, 96.4)
Routing:
- net Net-(U2-LA): track 15.3 -> 12.2 mm
- net Net-(U2-LB): track 19.9 -> 17.0 mm
- net GND: track 12.9 -> 10.1 mm, vias 0 -> 2
- net Net-(U2-RESETN): track 2.36 -> 1.32 mm

Commit message: update schematics and stuff
Parts:
- removed 11: ~, Library:25X48MM_NFC_EXPOSED_ANTENNA
- added D1: LED, LED_SMD:LED_0805_2012Metric, F.Cu at (142.3, 75.0)
- added D2: LED, LED_SMD:LED_0805_2012Metric, F.Cu at (146.1, 75.0)
- added D3: LED, LED_SMD:LED_0805_2012Metric, F.Cu at (149.9, 75.0)
- added D4: LED, LED_SMD:LED_0805_2012Metric, F.Cu at (153.8, 75.0)
- added J1: Conn_01x08_Pin, Library:8-Pin-Pads, F.Cu at (144.4, 109.0)
- added L1: ~, Library:25X48MM_NFC_EXPOSED_ANTENNA, F.Cu at (181.0, 95.2)
- added R1: R, Resistor_SMD:R_0201_0603Metric, F.Cu at (180.1, 113.2)
- moved C2 39.1 mm to (185.0, 109.9), turned to 90 degrees
- moved C3 38.3 mm to (185.2, 108.5), turned to 0 degrees
- moved C4 37.6 mm to (184.6, 113.0), turned to 0 degrees
- moved U2 31.9 mm to (181.5, 109.0), turned to 0 degrees
- moved C1 24.1 mm to (178.0, 108.2), turned to 90 degrees
Connections:
- net Net-(U2-RESETN) renamed /RESET
- net Net-(U2-VDDBAT) renamed VCC
- U2 pad 11: unconnected-(U2-PIO0_4/SCL-Pad11) -> /SCL
- U2 pad 12: unconnected-(U2-PIO0_5/SDA-Pad12) -> /SDA
- U2 pad 13: unconnected-(U2-PIO0_7/CT16B_M1-Pad13) -> /LEDC4
- U2 pad 15: unconnected-(U2-PIO0_10/CT32B_M0/SWCLK-Pad15) -> /SWCLK
- U2 pad 16: unconnected-(U2-PIO0_11/CT32B_M1/SWDIO-Pad16) -> /SWDIO
- U2 pad 2: unconnected-(U2-PIO0_1/CLKOUT-Pad2) -> /LEDR1
- U2 pad 4: unconnected-(U2-PIO0_6/SCLK-Pad4) -> /LEDC1
- U2 pad 5: unconnected-(U2-PIO0_8/MISO-Pad5) -> /LEDC2
- U2 pad 6: unconnected-(U2-PIO0_9/MOSI-Pad6) -> /LEDC3
Routing:
- net Net-(U2-LA): track 12.2 -> 19.5 mm, vias 0 -> 1
- net GND: track 10.1 -> 5.21 mm, vias 2 -> 0
- net /LEDR1: track 0.00 -> 3.89 mm, vias 0 -> 2
- net Net-(U2-PIO0_0/WAKEUP): track 1.50 -> 0.00 mm
- net Net-(U2-LB): track 17.0 -> 17.6 mm

Commit message: finish pcb routing
Parts:
- removed D4: LED, LED_SMD:LED_0805_2012Metric
- added REF**: HoldingHole, Library:HoldingHole, F.Cu at (124.5, 73.5)
- added REF**: Name_1, Library:Name_1, F.Cu at (129.5, 89.5)
- moved C4 68.6 mm to (116.0, 113.0), turned to 180 degrees
- moved R1 65.9 mm to (114.3, 109.5), turned to 90 degrees
- moved C2 62.0 mm to (123.0, 110.9)
- moved U2 62.0 mm to (119.5, 110.0)
- moved C1 61.4 mm to (116.6, 107.0), turned to 0 degrees
- moved C3 60.7 mm to (124.5, 110.0)
- moved D1 25.8 mm to (119.6, 87.2), turned to 45 degrees
- moved D2 25.1 mm to (122.7, 84.1), turned to 45 degrees
- moved D3 24.6 mm to (126.0, 80.8), turned to 45 degrees
Connections:
- C4 pad 1: Net-(U2-PIO0_0/WAKEUP) -> /WAKE
- J1 pad 3: /SWDIO -> /RESET
- J1 pad 5: /RESET -> /SWDIO
- J1 pad 6: VCC -> /WAKE
- U2 pad 1: Net-(U2-PIO0_0/WAKEUP) -> /WAKE
- U2 pad 13: /LEDC4 -> unconnected-(U2-PIO0_7/CT16B_M1-Pad13)
Routing:
- net /LEDC3: track 0.00 -> 46.4 mm, vias 0 -> 2
- net Net-(U2-LA): track 19.5 -> 64.1 mm
- net Net-(U2-LB): track 17.6 -> 58.8 mm
- net /LEDC2: track 0.00 -> 39.7 mm, vias 0 -> 2
- net /SCL: track 0.00 -> 37.6 mm, vias 0 -> 1
- net /WAKE: track 0.00 -> 36.7 mm, vias 0 -> 1
- net Net-(D1-A): track 0.00 -> 36.6 mm, vias 0 -> 2
- net /SDA: track 0.00 -> 34.1 mm, vias 0 -> 1
- net GND: track 5.21 -> 38.9 mm, vias 0 -> 1
- net /LEDC1: track 0.00 -> 31.7 mm, vias 0 -> 2
- net /SWDIO: track 0.00 -> 30.7 mm, vias 0 -> 1
- net /SWCLK: track 0.00 -> 28.0 mm, vias 0 -> 1
- net /RESET: track 1.70 -> 25.9 mm, vias 0 -> 1
- net VCC: track 1.55 -> 17.3 mm, vias 0 -> 1
- net /LEDR1: track 3.89 -> 7.86 mm

Commit message: stuff
Parts:
- added REF**: Wireless_icon, Library:Wireless_icon, F.Cu at (181.0, 95.0)
- added REF**: Position, Library:Position, F.Cu at (130.0, 96.5)
- added REF**: Contact, Library:Contact, F.Cu at (130.2, 97.0)
- moved J1 6.96 mm to (144.4, 116.0)
Routing:
- net /RESET: track 25.9 -> 30.3 mm
- net /SCL: track 37.6 -> 40.7 mm
- net /WAKE: track 36.7 -> 39.6 mm
- net /SDA: track 34.1 -> 36.5 mm
- net /SWDIO: track 30.7 -> 32.9 mm
- net /SWCLK: track 28.0 -> 29.8 mm
- net GND: track 38.9 -> 37.1 mm
- net VCC: track 17.3 -> 18.1 mm
Other:
- board text added: "GND"
- board text added: "VCC"

Commit message: stuff
Other:
- board text added: "RST"

Commit message: update footprints and stuff
Parts:
- moved J1 7.30 mm to (137.2, 114.5)
Routing:
- net /SCL: track 40.7 -> 51.3 mm
- net VCC: track 18.1 -> 12.1 mm
- net /WAKE: track 39.6 -> 44.1 mm
- net GND: track 37.1 -> 32.8 mm
- net /SDA: track 36.5 -> 38.7 mm
- net /SWDIO: track 32.9 -> 34.1 mm
- net /RESET: track 30.3 -> 29.2 mm
- net /SWCLK: track 29.8 -> 29.2 mm
Other:
- board text added: "SCL"
- board text added: "SDL"
- board text added: "SWCLK"
- board text added: "SWDIO"
- board text added: "WAKE"

Commit message: finalize pcb
Parts:
- R1: value R -> 330
- moved R1 0.41 mm to (114.8, 109.5)
Routing:
- net /SWDIO: track 34.1 -> 35.5 mm
- net /SWCLK: track 29.2 -> 30.3 mm
- net /SCL: track 51.3 -> 50.7 mm
Other:
- board text added: "RESET"
- board text added: "SDA"
- board text removed: "RST"
- board text removed: "SDL"

Commit message: business card stuff
Parts:
- C2, C3, C4: footprint Capacitor_SMD:C_0201_0603Metric -> Capacitor_SMD:C_0402_1005Metric
- D1, D2, D3: footprint LED_SMD:LED_0805_2012Metric -> LED_SMD:LED_1206_3216Metric
- R1: footprint Resistor_SMD:R_0201_0603Metric -> Resistor_SMD:R_0402_1005Metric
- moved R1 69.4 mm to (184.1, 109.4), turned to 45 degrees
- moved C4 68.9 mm to (184.9, 111.5), turned to -90 degrees
- moved C1 66.5 mm to (182.6, 115.0), turned to -90 degrees
- moved U2 61.5 mm to (181.0, 111.5), turned to 135 degrees
- moved C2 56.6 mm to (179.6, 108.3), turned to -135 degrees
- moved C3 52.8 mm to (177.3, 108.4), turned to 135 degrees
- moved REF** 1.60 mm to (131.2, 95.8)
- moved REF** 1.52 mm to (131.0, 89.2)
- moved REF** 1.35 mm to (131.2, 96.0)
- moved D1 0.37 mm to (119.3, 87.4)
- moved REF** 0.20 mm to (181.0, 95.2)
- renumbered REF** to H1
Connections:
- U2 pad 4: /LEDC1 -> /LEDC3
- U2 pad 6: /LEDC3 -> /LEDC1
Routing:
- net GND: track 33.2 -> 149.0 mm, vias 1 -> 4
- net /LEDC1: track 31.7 -> 83.9 mm
- net Net-(D1-A): track 36.3 -> 87.9 mm
- net VCC: track 12.1 -> 55.1 mm
- net /LEDC2: track 39.7 -> 81.0 mm
- net Net-(U2-LA): track 64.1 -> 25.6 mm
- net /LEDC3: track 46.4 -> 78.2 mm
- net Net-(U2-LB): track 58.8 -> 30.1 mm
- net /SCL: track 50.7 -> 25.5 mm
- net /RESET: track 29.2 -> 45.3 mm
- net /SWCLK: track 30.3 -> 42.3 mm
- net /SDA: track 38.7 -> 28.7 mm
- net /LEDR1: track 8.03 -> 1.41 mm, vias 2 -> 0
- net /SWDIO: track 35.5 -> 39.7 mm
- net /WAKE: track 44.1 -> 46.8 mm
Other:
- board text added: "-. . .-. -.."
- board text added: "evanyu.dev"
- board text added: "github.com/Badbird5907"
- board text added: "linkedin.com/in/badbird"
- board text added: "twitter.com/Badbird5907"
